File: ESP32WROVERSNAP/ESP32WROVERSNAP.kicad_pcb (KiCad board)
At the start: 2 copper layers, 50 x 50.5 mm, 35 parts, among them IC2 RESET, IC3 BOOT, IC4 ESP32-Wrover-IE-N16R8, IC5 5PB1102, J1 Conn_01x09_Socket, J2 PROG, J3 POWER IN, J4 I2S OUT, J5 Conn_01x09_Socket, U1 LD1117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

Commit message: ?
Parts:
- removed C10, C12, C5: 100nF, Capacitor_SMD:C_1206_3216Metric_Pad1.33x1.80mm_HandSolder
- removed IC5: 5PB1102, Custom:5PB1102PGGK
- removed R10: 270K, Resistor_SMD:R_0805_2012Metric_Pad1.20x1.40mm_HandSolder
- removed R11: 47K, Resistor_SMD:R_0805_2012Metric_Pad1.20x1.40mm_HandSolder
- removed R12, R9: 10K, Resistor_SMD:R_0603_1608Metric_Pad0.98x0.95mm_HandSolder
- removed R13, R14: 22R, Resistor_SMD:R_0805_2012Metric_Pad1.20x1.40mm_HandSolder
- removed Y2: 22.5792MHz, Oscillator:Oscillator_SMD_Abracon_ASE-4Pin_3.2x2.5mm
- added G***: LOGO, Custom:LOGONEW, F.Cu at (170.3, 66.8)
- added R6: 0R*, Resistor_SMD:R_0805_2012Metric_Pad1.20x1.40mm_HandSolder, F.Cu at (140.0, 67.6)
Connections:
- J1 pad 9: /SENSEIN -> unconnected-(J1-Pin_9-Pad9)
Routing:
- net /SENSEIN: track 31.2 -> 0.00 mm, vias 1 -> 0
- net /SENSE: track 21.5 -> 0.00 mm
- net /3V3: track 129.8 -> 136.5 mm
- net /5V: track 72.2 -> 76.5 mm
- net GND: vias 25 -> 42
Other:
- board text added: "NC BCK DATA LRCK GND GND"
- board text removed: "SCK BCK DATA LRCK GND GND"
