File: ESP32WROVERSNAP/ESP32WROVERSNAP.kicad_sch (KiCad schematic)
At the start: 35 parts, among them IC2 RESET, IC3 BOOT, IC4 ESP32-Wrover-IE-N16R8, IC5 5PB1102, J1 Conn_01x09_Socket, J2 PROG, J3 POWER IN, J4 I2S OUT, J5 Conn_01x09_Socket, U1 LD1117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

Commit message: ?
Parts:
- removed C10, C12, C5: 100nF, Capacitor_SMD:C_1206_3216Metric_Pad1.33x1.80mm_HandSolder, symbol Device:C
- removed IC5: 5PB1102, Custom:5PB1102PGGK, symbol Custom:5PB1102PGGK
- removed R10: 270K, Resistor_SMD:R_0805_2012Metric_Pad1.20x1.40mm_HandSolder, symbol Device:R
- removed R11: 47K, Resistor_SMD:R_0805_2012Metric_Pad1.20x1.40mm_HandSolder, symbol Device:R
- removed R12, R9: 10K, Resistor_SMD:R_0603_1608Metric_Pad0.98x0.95mm_HandSolder, symbol Device:R
- removed R13, R14: 22R, Resistor_SMD:R_0805_2012Metric_Pad1.20x1.40mm_HandSolder, symbol Device:R
- removed Y2: 22.5792MHz, Oscillator:Oscillator_SMD_Abracon_ASE-4Pin_3.2x2.5mm, symbol Oscillator:ASE-xxxMHz
- added R6: 0R*, Resistor_SMD:R_0805_2012Metric_Pad1.20x1.40mm_HandSolder, symbol Device:R
Connections:
- net 3V3: now also R6.2
- net 5V: now also R6.1
- net SENSEIN: no longer names the net of J1.9 (Pin_9)
